File: nRF9161-DEV-BOARD.kicad_pcb (KiCad board)
At the start: 4 copper layers, 120 x 80 mm, 103 parts, among them J1 VIN_3V0-5V5, J10 SPI0, J11 I2C0, J12 GPIO_P0.00-15, J13 GPIO_P0.16-31, J14 RFFE_MAGPIO, J15 COEX, J16 I2S, J17 PDM, J18 ADC_AIN0-7, J2 U.FL_LTE_NR+, J3 SWF_LTE, J5 U.FL_GNSS, J6 SWF_GNSS, J7 nanoSIM_4FF, J8 SWD_10pin, J9 UART0, SW1 DISABLE, SW2 RESET, SW3 USER, U1 NRF9161-LACA-R7, U2 TLV73330PDBV, U3 TPS22919DCKR, U4 TPD3F303DPV

Commit message: PCB pass30an KEEP: VDD_GPIO opens 2→1; unconnected still 63 (offset by waived GND island 11→12); D3.1 clearance 0.385 mm; short/clearance/crossing/hole 0; hole_to_hole 1
Routing:
- net VDD_GPIO: track 415.3 -> 443.4 mm
Changed lines of the file:
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@@
+	)
+	(segment
+		(start 77.3 7.05)
+		(end 81.5 13.5)
+		(width 0.18)
+		(layer "F.Cu")
+		(net 22)
 	)
 	(segment
@@
 	)
 	(segment
+		(start 81.5 13.5)
+		(end 86.51 26)
+		(width 0.18)
+		(layer "F.Cu")
+		(net 22)
+	)
+	(segment
 		(start 46.64 76)
 		(end 49.18 76)
@@
 	)
 	(segment
+		(start 71.3 8)
+		(end 71.3 7.05)
+		(width 0.18)
+		(layer "F.Cu")
+		(net 22)
+	)
+	(segment
 		(start 39.52 19.125833)
 		(end 40.17 19.125833)
@@
 		(layer "F.Cu")
 		(net 22)
+	)
+	(segment
+		(start 71.3 7.05)
+		(end 77.3 7.05)
+		(width 0.18)
+		(layer "F.Cu")
+		(net 22)

Commit message: PCB pass30ap KEEP: VDD_GPIO opens 1→0; unconnected 63→62; GND islands 12; short/clearance/crossing/hole 0; hole_to_hole 1; tightest foreign clearance 0.207 mm to SIM_CLK
Routing:
- net VDD_GPIO: track 443.4 -> 484.7 mm
Changed lines of the file:
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@@
+	)
+	(segment
+		(start 76.4375 41.55)
+		(end 74.438 43.05)
+		(width 0.18)
+		(layer "F.Cu")
+		(net 22)
 	)
 	(segment
@@
 	)
 	(segment
+		(start 70.438 41.55)
+		(end 54.438 61.05)
+		(width 0.18)
+		(layer "F.Cu")
+		(net 22)
+	)
+	(segment
 		(start 40.17 20.2)
 		(end 45.9 20.2)
@@
 	)
 	(segment
+		(start 71.938 42.05)
+		(end 70.438 41.55)
+		(width 0.18)
+		(layer "F.Cu")
+		(net 22)
+	)
+	(segment
 		(start 104 67.08)
 		(end 105.1 67.08)
@@
 	)
 	(segment
+		(start 76.4375 39.05)
+		(end 76.4375 41.55)
+		(width 0.18)
+		(layer "F.Cu")
+		(net 22)
+	)
+	(segment
 		(start 78 32)
 		(end 79.3 32)
@@
 	)
 	(segment
+		(start 74.438 43.05)
+		(end 72.438 43.05)
+		(width 0.18)
+		(layer "F.Cu")
+		(net 22)
+	)
+	(segment
 		(start 48.05 3.46)
 		(end 46.349999 3.46)
@@
 	)
 	(segment
+		(start 54.438 63.55)
+		(end 58.2 62.7)
+		(width 0.18)
+		(layer "F.Cu")
+		(net 22)
+	)
+	(segment
 		(start 114.4 38.16)
 		(end 114.4 31.08)
@@
 	)
 	(segment
+		(start 72.438 43.05)
+		(end 71.938 42.05)
+		(width 0.18)
+		(layer "F.Cu")
+		(net 22)
+	)
+	(segment
 		(start 71.3 7.05)
 		(end 77.3 7.05)
@@
 		(width 0.18)
 		(layer "F.Cu")
+		(net 22)
+	)
+	(segment
+		(start 54.438 61.05)
+		(end 54.438 63.55)
+		(width 0.18)
+		(layer "F.Cu")

Commit message: PCB pass30aq KEEP: P0.31 header-to-header; opens 2→1; unconnected 62→61; GND islands 12; short/clearance/crossing/hole 0; hole_to_hole 1; foreign 0.230 mm; POWER 0.245 mm
Routing:
- net P0.31: track 0.00 -> 46.2 mm
Changed lines of the file:
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@@
+	)
+	(segment
+		(start 103.05 47.1)
+		(end 106.7 47.1)
+		(width 0.18)
+		(layer "F.Cu")
+		(net 16)
+	)
+	(segment
+		(start 102.6 75.5)
+		(end 103.05 47.1)
+		(width 0.18)
+		(layer "F.Cu")
+		(net 16)
+	)
+	(segment
+		(start 114.9 50.62)
+		(end 114.9 48.8)
+		(width 0.18)
+		(layer "F.Cu")
+		(net 16)
+	)
+	(segment
+		(start 106.7 50.62)
+		(end 114.9 50.62)
+		(width 0.18)
+		(layer "F.Cu")
+		(net 16)
+	)
+	(segment
+		(start 106.7 47.1)
+		(end 106.7 50.62)
+		(width 0.18)
+		(layer "F.Cu")
+		(net 16)
+	)
+	(segment
+		(start 114.9 48.8)
+		(end 115.55 48.8)
+		(width 0.18)
+		(layer "F.Cu")
+		(net 16)
 	)
 	(segment

Commit message: PCB pass30as KEEP: P0.30 header-to-header; opens 2→1; unconnected 61→60; GND islands 12; short/clearance/crossing/hole 0; hole_to_hole 1; foreign 0.29 mm; POWER 0.70 mm
Routing:
- net P0.30: track 3.85 -> 54.1 mm, vias 1 -> 2
Changed lines of the file:
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@@
+	)
+	(segment
+		(start 99.56 75.28)
+		(end 99.56 74.7)
+		(width 0.18)
+		(layer "F.Cu")
+		(net 35)
+	)
+	(segment
+		(start 101.2 46.4)
+		(end 112.4 46.4)
+		(width 0.18)
+		(layer "F.Cu")
+		(net 35)
+	)
+	(segment
+		(start 101.2 74.7)
+		(end 101.2 46.4)
+		(width 0.18)
+		(layer "F.Cu")
+		(net 35)
+	)
+	(segment
+		(start 99.56 74.7)
+		(end 101.2 74.7)
+		(width 0.18)
+		(layer "F.Cu")
+		(net 35)
 	)
 	(segment
@@
 	)
 	(via
+		(at 112.4 46.4)
+		(size 0.6)
+		(drill 0.3)
+		(layers "F.Cu" "B.Cu")
+		(net 35)
+	)
+	(via
 		(at 36.25 41.1)
 		(size 0.6)
@@
 		(net 35)
 	)
+	(segment
+		(start 117.6 45)
+		(end 117.6 46)
+		(width 0.18)
+		(layer "B.Cu")
+		(net 35)
+	)
+	(segment
+		(start 112.4 46.4)
+		(end 112.4 45)
+		(width 0.18)
+		(layer "B.Cu")
+		(net 35)
+	)
+	(segment
+		(start 117.6 46)
+		(end 116.7 46)
+		(width 0.18)
+		(layer "B.Cu")
+		(net 35)
+	)
+	(segment
+		(start 112.4 45)
+		(end 117.6 45)
+		(width 0.18)
+		(layer "B.Cu")
+		(net 35)
+	)

Commit message: PCB pass30ax KEEP: P0.16 closed (In1 skirt via 40.70,20.80 to J18.4); opens 1→0; 60→59; GND islands 12; foreign 0.21 mm; POWER 0.338 mm; short/clr/cross/hole 0; hole_to_hole 1
Routing:
- net P0.16: track 70.7 -> 117.9 mm
Changed lines of the file:
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@@
+	)
+	(segment
+		(start 40.7 20.8)
+		(end 45.55 20.8)
+		(width 0.18)
+		(layer "In1.Cu")
+		(net 9)
+	)
+	(segment
+		(start 44.6 60.4)
+		(end 45.62 60.4)
+		(width 0.18)
+		(layer "In1.Cu")
+		(net 9)
+	)
+	(segment
+		(start 44.6 27.4)
+		(end 44.6 60.4)
+		(width 0.18)
+		(layer "In1.Cu")
+		(net 9)
+	)
+	(segment
+		(start 45.55 27.4)
+		(end 44.6 27.4)
+		(width 0.18)
+		(layer "In1.Cu")
+		(net 9)
+	)
+	(segment
+		(start 45.62 60.4)
+		(end 45.62 61.1)
+		(width 0.18)
+		(layer "In1.Cu")
+		(net 9)
+	)
+	(segment
+		(start 45.55 20.8)
+		(end 45.55 27.4)
+		(width 0.18)
+		(layer "In1.Cu")
+		(net 9)
 	)
 	(segment

Commit message: PCB pass30ay KEEP: P0.17 closed (In2 skirt via 40.25,23.10 to J18.5); opens 2→1; 59→58; GND islands 12; foreign 0.21 mm; POWER 0.338 mm; short/clr/cross/hole 0; hole_to_hole 1
Routing:
- net P0.17: track 71.2 -> 122.4 mm
Changed lines of the file:
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@@
+	)
+	(segment
+		(start 40.25 23.1)
+		(end 40.25 21.5)
+		(width 0.18)
+		(layer "In2.Cu")
+		(net 11)
+	)
+	(segment
+		(start 48.16 60.4)
+		(end 48.16 61.3)
+		(width 0.18)
+		(layer "In2.Cu")
+		(net 11)
+	)
+	(segment
+		(start 45.55 21.5)
+		(end 45.55 27.4)
+		(width 0.18)
+		(layer "In2.Cu")
+		(net 11)
+	)
+	(segment
+		(start 40.25 21.5)
+		(end 45.55 21.5)
+		(width 0.18)
+		(layer "In2.Cu")
+		(net 11)
+	)
+	(segment
+		(start 44.6 60.4)
+		(end 48.16 60.4)
+		(width 0.18)
+		(layer "In2.Cu")
+		(net 11)
+	)
+	(segment
+		(start 44.6 27.4)
+		(end 44.6 60.4)
+		(width 0.18)
+		(layer "In2.Cu")
+		(net 11)
+	)
+	(segment
+		(start 45.55 27.4)
+		(end 44.6 27.4)
+		(width 0.18)
+		(layer "In2.Cu")
+		(net 11)
 	)
 	(segment
