File: panel/nRF9161-v2-panel.kicad_pcb (KiCad board)
At the start: 4 copper layers, 118 x 93 mm, 474 parts, among them J2 U.FL_LTE_NR+, J20 HOST_1x10_2.54, J5 U.FL_GNSS, J7 nanoSIM_4FF, J8 SWD_10pin, Q1 BSS138, SW2 RESET, U1 NRF9161-LACA-R7, U2 TLV73333PDBV, U3 TPS22919DCKR, U4 TPD3F303DPV, U5 SN74LXC2T45, U6 SN74LXC2T45, U7 SN74LXC1T45, U8 SN74LXC1T45

Commit message: v2 fab pass 5ad8bde: RED (21 silk labels 0.8 mm < 1.0 mm JLC min); 22/88 filled vias; panel rebuilt (stale silk); package fab/staging-v2-5ad8bde
Parts:
- moved KiKit_MB_13_1 50.0 mm to (159.5, 105.1)
- moved KiKit_MB_13_2 50.0 mm to (158.5, 105.1)
- moved KiKit_MB_13_3 50.0 mm to (157.5, 105.1)
- moved KiKit_MB_13_4 50.0 mm to (156.5, 105.1)
- moved KiKit_MB_13_5 50.0 mm to (155.5, 105.1)
- moved KiKit_MB_1_1 50.0 mm to (107.5, 65.6)
- moved KiKit_MB_1_2 50.0 mm to (106.5, 65.6)
- moved KiKit_MB_1_3 50.0 mm to (105.5, 65.6)
- moved KiKit_MB_1_4 50.0 mm to (104.5, 65.6)
- moved KiKit_MB_1_5 50.0 mm to (103.5, 65.6)
- moved KiKit_MB_5_1 50.0 mm to (159.5, 65.6)
- moved KiKit_MB_5_2 50.0 mm to (158.5, 65.6)
- moved KiKit_MB_5_3 50.0 mm to (157.5, 65.6)
- moved KiKit_MB_5_4 50.0 mm to (156.5, 65.6)
- moved KiKit_MB_5_5 50.0 mm to (155.5, 65.6)
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Other:
- outline, holes or cut-outs redrawn
