File: schematic/03_LTE_RF.kicad_sch (KiCad schematic)
At the start: 11 parts, among them J14 RFFE_MAGPIO, J15 COEX, J2 U.FL_LTE_NR+, J3 SWF_LTE

Commit message: Schematic: GNSS COEX0 bias switch, 3.3V VDD_GPIO, DNP RF shunts
- Add U3 TPS22919DCKR on 04_GNSS (COEX0-gated bias); FB5 0402
- Swap U2 to TLV73333 (3.3 V VDD_GPIO); DNP Class-C shunt caps
- Quarantine leftover schematics/; remove stale ERC rpt
- Add PM/DFM/RF/schematic/layout review docs under docs/
Parts:
- C21, C22, C23, C24: now not fitted; now left out of the parts list
Changed lines of the file:
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@@
 		(unit 1)
 		(exclude_from_sim no)
-		(in_bom yes)
-		(on_board yes)
-		(dnp no)
+		(in_bom no)
+		(on_board yes)
+		(dnp yes)
 		(property "Reference" "C21"
 			(at 50.8 60.96 0)
@@
 		(unit 1)
 		(exclude_from_sim no)
-		(in_bom yes)
-		(on_board yes)
-		(dnp no)
+		(in_bom no)
+		(on_board yes)
+		(dnp yes)
 		(property "Reference" "C22"
 			(at 76.2 60.96 0)
@@
 		(unit 1)
 		(exclude_from_sim no)
-		(in_bom yes)
-		(on_board yes)
-		(dnp no)
+		(in_bom no)
+		(on_board yes)
+		(dnp yes)
 		(property "Reference" "C23"
 			(at 50.8 124.46 0)
@@
 		(unit 1)
 		(exclude_from_sim no)
-		(in_bom yes)
-		(on_board yes)
-		(dnp no)
+		(in_bom no)
+		(on_board yes)
+		(dnp yes)
 		(property "Reference" "C24"
 			(at 76.2 124.46 0)

Commit message: Exclude JP1, JP2, TP1-TP20 from BOM (attrs only, sch+pcb)
Parts:
- TP1: now left out of the parts list
Changed lines of the file:
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@@
 		(unit 1)
 		(exclude_from_sim no)
-		(in_bom yes)
+		(in_bom no)
 		(on_board yes)
 		(dnp no)

Commit message: v2: simplify to UART modem module (J20 host header, LXC translators); remove J1, J3, J6, J9-J18, optional parts
Parts:
- removed J14: RFFE_MAGPIO, Connector_PinHeader_1.27mm:PinHeader_1x06_P1.27mm_Vertical, symbol Connector_Generic:Conn_01x06
- removed J15: COEX, Connector_PinHeader_1.27mm:PinHeader_1x06_P1.27mm_Vertical, symbol Connector_Generic:Conn_01x06
- removed J3: SWF_LTE, Board:Murata_MM8130-2600_SWF, symbol Connector:Conn_Coaxial

Commit message: v2 BOM: apply footprint-consistent MPNs + LCSC IDs, JLC BOM, audit reports (U4 footprint pending Layout)
Parts:
- J2: LCSC (none) -> C88373; MPN (none) -> U.FL-R-SMT-1(10); Manufacturer (none) -> Hirose
- L1, L2: value 0R / DNP match -> 0R; LCSC (none) -> C17168; MPN (none) -> 0402WGF0000TCE; Manufacturer (none) -> UNI-ROYAL
Changed lines of the file:
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@@
 			)
 		)
-		(property "Value" "0R / DNP match"
+		(property "Value" "0R"
 			(at 63.5 53.34 0)
 			(show_name no)
@@
 			(show_name no)
 			(do_not_autoplace no)
+			(effects
+				(font
+					(size 1.27 1.27)
+				)
+			)
+		)
+		(property "MPN" "0402WGF0000TCE"
+			(at 63.5 50.8 90)
+			(hide yes)
+			(effects
+				(font
+					(size 1.27 1.27)
+				)
+			)
+		)
+		(property "LCSC" "C17168"
+			(at 63.5 50.8 90)
+			(hide yes)
+			(effects
+				(font
+					(size 1.27 1.27)
+				)
+			)
+		)
+		(property "Manufacturer" "UNI-ROYAL"
+			(at 63.5 50.8 90)
+			(hide yes)
 			(effects
 				(font
@@
 			)
 		)
+		(property "MPN" "U.FL-R-SMT-1(10)"
+			(at 101.6 50.8 0)
+			(hide yes)
+			(effects
+				(font
+					(size 1.27 1.27)
+				)
+			)
+		)
+		(property "LCSC" "C88373"
+			(at 101.6 50.8 0)
+			(hide yes)
+			(effects
+				(font
+					(size 1.27 1.27)
+				)
+			)
+		)
+		(property "Manufacturer" "Hirose"
+			(at 101.6 50.8 0)
+			(hide yes)
+			(effects
+				(font
+					(size 1.27 1.27)
+				)
+			)
+		)
 		(pin "1"
 		)
@@
 			)
 		)
-		(property "Value" "0R / DNP match"
+		(property "Value" "0R"
 			(at 63.5 116.84 0)
 			(show_name no)
@@
 			(effects
 				(font
+					(size 1.27 1.27)
+				)
+			)
+		)
+		(property "MPN" "0402WGF0000TCE"
+			(at 63.5 114.3 90)
+			(hide yes)
+			(effects
+				(font
+					(size 1.27 1.27)
+				)
+			)
+		)
+		(property "LCSC" "C17168"
+			(at 63.5 114.3 90)
+			(hide yes)
+			(effects
+				(font
+					(size 1.27 1.27)
+				)
+			)
+		)
+		(property "Manufacturer" "UNI-ROYAL"
+			(at 63.5 114.3 90)
+			(hide yes)
+			(effects
+				(font
