File: schematic/11_LEDS_BUTTONS.kicad_sch (KiCad schematic)
At the start: 10 parts, among them SW3 USER

Commit message: Schematic: add C40 100nF X7R on SIM_1V8 at U1; D3-D7 values restored (Function field); D7 DNP; ERC 0 errors
Parts:
- D4: value STATUS -> Green LED; Function (none) -> STATUS; MPN (none) -> KP-2012SGC; Manufacturer (none) -> Kingbright
- D5: value LTE -> Green LED; Function (none) -> LTE; MPN (none) -> KP-2012SGC; Manufacturer (none) -> Kingbright
- D6: value GNSS -> Green LED; Function (none) -> GNSS; MPN (none) -> KP-2012SGC; Manufacturer (none) -> Kingbright
- D7: value SPARE_DNP -> Green LED; Function Optional spare LED on P0.03; leave unpopulated to free GPIO -> SPARE_DNP; MPN (none) -> KP-2012SGC; Manufacturer (none) -> Kingbright; Note (none) -> Optional spare LED on P0.03; leave unpopulated to free GPIO; now not fitted; now left out of the parts list
Changed lines of the file:
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@@
 			)
 		)
-		(property "Value" "STATUS"
+		(property "Value" "Green LED"
 			(at 76.2 40.64 0)
+			(show_name no)
+			(do_not_autoplace no)
+			(effects
+				(font
+					(size 1.27 1.27)
+				)
+			)
+		)
+		(property "Function" "STATUS"
+			(at 76.2 43.18 0)
+			(show_name no)
+			(do_not_autoplace no)
+			(effects
+				(font
+					(size 1.27 1.27)
+				)
+			)
+		)
+		(property "Manufacturer" "Kingbright"
+			(at 76.2 40.64 0)
+			(hide yes)
+			(show_name no)
+			(do_not_autoplace no)
+			(effects
+				(font
+					(size 1.27 1.27)
+				)
+			)
+		)
+		(property "MPN" "KP-2012SGC"
+			(at 76.2 40.64 0)
+			(hide yes)
 			(show_name no)
 			(do_not_autoplace no)
@@
 			)
 		)
-		(property "Value" "LTE"
+		(property "Value" "Green LED"
 			(at 76.2 66.04 0)
+			(show_name no)
+			(do_not_autoplace no)
+			(effects
+				(font
+					(size 1.27 1.27)
+				)
+			)
+		)
+		(property "Function" "LTE"
+			(at 76.2 68.58 0)
+			(show_name no)
+			(do_not_autoplace no)
+			(effects
+				(font
+					(size 1.27 1.27)
+				)
+			)
+		)
+		(property "Manufacturer" "Kingbright"
+			(at 76.2 66.04 0)
+			(hide yes)
+			(show_name no)
+			(do_not_autoplace no)
+			(effects
+				(font
+					(size 1.27 1.27)
+				)
+			)
+		)
+		(property "MPN" "KP-2012SGC"
+			(at 76.2 66.04 0)
+			(hide yes)
 			(show_name no)
 			(do_not_autoplace no)
@@
 			)
 		)
-		(property "Value" "GNSS"
+		(property "Value" "Green LED"
 			(at 76.2 91.44 0)
+			(show_name no)
+			(do_not_autoplace no)
+			(effects
+				(font
+					(size 1.27 1.27)
+				)
+			)
+		)
+		(property "Function" "GNSS"
+			(at 76.2 93.98 0)
+			(show_name no)
+			(do_not_autoplace no)
+			(effects
+				(font
+					(size 1.27 1.27)
+				)
+			)
+		)
+		(property "Manufacturer" "Kingbright"
+			(at 76.2 91.44 0)
+			(hide yes)
+			(show_name no)
+			(do_not_autoplace no)
+			(effects
+				(font
+					(size 1.27 1.27)
+				)
+			)
+		)
+		(property "MPN" "KP-2012SGC"
+			(at 76.2 91.44 0)
+			(hide yes)
 			(show_name no)
 			(do_not_autoplace no)
@@
 		(unit 1)
 		(exclude_from_sim no)
-		(in_bom yes)
+		(in_bom no)
 		(on_board yes)
-		(dnp no)
+		(dnp yes)
 		(property "Reference" "D7"
 			(at 76.2 111.76 0)
@@
 			)
 		)
-		(property "Value" "SPARE_DNP"
+		(property "Value" "Green LED"
 			(at 76.2 116.84 0)
+			(show_name no)
+			(do_not_autoplace no)
+			(effects
+				(font
+					(size 1.27 1.27)
+				)
+			)
+		)
+		(property "Function" "SPARE_DNP"
+			(at 76.2 119.38 0)
+			(show_name no)
+			(do_not_autoplace no)
+			(effects
+				(font
+					(size 1.27 1.27)
+				)
+			)
+		)
+		(property "Manufacturer" "Kingbright"
+			(at 76.2 116.84 0)
+			(hide yes)
+			(show_name no)
+			(do_not_autoplace no)
+			(effects
+				(font
+					(size 1.27 1.27)
+				)
+			)
+		)
+		(property "MPN" "KP-2012SGC"
+			(at 76.2 116.84 0)
+			(hide yes)
 			(show_name no)
 			(do_not_autoplace no)
@@
       (effects (font (size 1.27 1.27)) (hide yes))
     )
-    (property "Function" "Optional spare LED on P0.03; leave unpopulated to free GPIO" (at 76.2 114.3 0)
+    (property "Note" "Optional spare LED on P0.03; leave unpopulated to free GPIO" (at 76.2 114.3 0)
       (effects (font (size 1.27 1.27)) (hide yes))
     )

Commit message: v2: simplify to UART modem module (J20 host header, LXC translators); remove J1, J3, J6, J9-J18, optional parts
Parts:
- removed D5, D6, D7: Green LED, LED_SMD:LED_0603_1608Metric, symbol Device:LED
- removed R11, R12, R13: 1k, Resistor_SMD:R_0402_1005Metric, symbol Device:R
- removed R14: 10k, Resistor_SMD:R_0402_1005Metric, symbol Device:R
- removed SW3: USER, Button_Switch_SMD:SW_SPST_CK_KXT3, symbol Switch:SW_Push

Commit message: v2 BOM: apply footprint-consistent MPNs + LCSC IDs, JLC BOM, audit reports (U4 footprint pending Layout)
Parts:
- D4: LCSC (none) -> C125098; MPN KP-2012SGC -> LTST-C191KGKT; Manufacturer Kingbright -> Lite-On
- R10: LCSC (none) -> C11702; MPN (none) -> 0402WGF1001TCE; Manufacturer (none) -> UNI-ROYAL
Changed lines of the file:
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@@
 			)
 		)
-		(property "Manufacturer" "Kingbright"
+		(property "Manufacturer" "Lite-On"
 			(at 76.2 40.64 0)
 			(hide yes)
@@
 			)
 		)
-		(property "MPN" "KP-2012SGC"
+		(property "MPN" "LTST-C191KGKT"
 			(at 76.2 40.64 0)
 			(hide yes)
@@
 			(show_name no)
 			(do_not_autoplace no)
+			(effects
+				(font
+					(size 1.27 1.27)
+				)
+			)
+		)
+		(property "LCSC" "C125098"
+			(at 76.2 38.1 0)
+			(hide yes)
 			(effects
 				(font
@@
 			(effects
 				(font
+					(size 1.27 1.27)
+				)
+			)
+		)
+		(property "MPN" "0402WGF1001TCE"
+			(at 50.8 38.1 90)
+			(hide yes)
+			(effects
+				(font
+					(size 1.27 1.27)
+				)
+			)
+		)
+		(property "LCSC" "C11702"
+			(at 50.8 38.1 90)
+			(hide yes)
+			(effects
+				(font
+					(size 1.27 1.27)
+				)
+			)
+		)
+		(property "Manufacturer" "UNI-ROYAL"
+			(at 50.8 38.1 90)
+			(hide yes)
+			(effects
+				(font
