File: schematic/05_SIM.kicad_sch (KiCad schematic)
At the start: 13 parts, among them J7 nanoSIM_4FF, U4 TPD3F303DPV

Commit message: Exclude JP1, JP2, TP1-TP20 from BOM (attrs only, sch+pcb)
Parts:
- JP2, TP3, TP4, TP5, TP6: now left out of the parts list
Changed lines of the file:
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@@
 		(unit 1)
 		(exclude_from_sim no)
-		(in_bom yes)
+		(in_bom no)
 		(on_board yes)
 		(dnp no)
@@
 		(unit 1)
 		(exclude_from_sim no)
-		(in_bom yes)
+		(in_bom no)
 		(on_board yes)
 		(dnp no)
@@
 		(unit 1)
 		(exclude_from_sim no)
-		(in_bom yes)
+		(in_bom no)
 		(on_board yes)
 		(dnp no)
@@
 		(unit 1)
 		(exclude_from_sim no)
-		(in_bom yes)
+		(in_bom no)
 		(on_board yes)
 		(dnp no)
@@
 		(unit 1)
 		(exclude_from_sim no)
-		(in_bom yes)
-		(on_board yes)
-		(dnp no)
+		(in_bom no)
+		(on_board yes)
+		(dnp no)

Commit message: v2: simplify to UART modem module (J20 host header, LXC translators); remove J1, J3, J6, J9-J18, optional parts
Parts:
- removed TP3: SIM_CLK, TestPoint:TestPoint_Pad_D1.0mm, symbol Connector:TestPoint
- removed TP4: SIM_RST, TestPoint:TestPoint_Pad_D1.0mm, symbol Connector:TestPoint
- removed TP5: SIM_IO, TestPoint:TestPoint_Pad_D1.0mm, symbol Connector:TestPoint
- removed TP6: SIM_CD, TestPoint:TestPoint_Pad_D1.0mm, symbol Connector:TestPoint

Commit message: v2 BOM: apply footprint-consistent MPNs + LCSC IDs, JLC BOM, audit reports (U4 footprint pending Layout)
Parts:
- C33: LCSC (none) -> C1525; MPN (none) -> CL05B104KO5NNNC; Manufacturer (none) -> Samsung Electro-Mechanics
- C34: LCSC (none) -> C16772; MPN (none) -> CL05B224KO5NNNC; Manufacturer (none) -> Samsung Electro-Mechanics
- C35, C36, C37, C38: LCSC (none) -> C76924; MPN (none) -> GRM0335C1H220JA01D; Manufacturer (none) -> Murata
- J7: LCSC (none) -> C2977286; MPN (none) -> SF72S006VBDR2500; Manufacturer (none) -> JAE
- U4: LCSC (none) -> C2865991; MPN (none) -> TPD3F303DPVR; Manufacturer (none) -> Texas Instruments
Changed lines of the file:
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@@
+			)
+		)
+		(property "MPN" "SF72S006VBDR2500"
+			(at 101.6 63.5 0)
+			(hide yes)
+			(effects
+				(font
+					(size 1.27 1.27)
+				)
+			)
+		)
+		(property "LCSC" "C2977286"
+			(at 101.6 63.5 0)
+			(hide yes)
+			(effects
+				(font
+					(size 1.27 1.27)
+				)
+			)
+		)
+		(property "Manufacturer" "JAE"
+			(at 101.6 63.5 0)
+			(hide yes)
+			(effects
+				(font
+					(size 1.27 1.27)
+				)
 			)
 		)
@@
 			)
 		)
+		(property "MPN" "TPD3F303DPVR"
+			(at 50.8 63.5 0)
+			(hide yes)
+			(effects
+				(font
+					(size 1.27 1.27)
+				)
+			)
+		)
+		(property "LCSC" "C2865991"
+			(at 50.8 63.5 0)
+			(hide yes)
+			(effects
+				(font
+					(size 1.27 1.27)
+				)
+			)
+		)
+		(property "Manufacturer" "Texas Instruments"
+			(at 50.8 63.5 0)
+			(hide yes)
+			(effects
+				(font
+					(size 1.27 1.27)
+				)
+			)
+		)
 		(pin "1"
 		)
@@
 			)
 		)
+		(property "MPN" "CL05B104KO5NNNC"
+			(at 50.8 101.6 0)
+			(hide yes)
+			(effects
+				(font
+					(size 1.27 1.27)
+				)
+			)
+		)
+		(property "LCSC" "C1525"
+			(at 50.8 101.6 0)
+			(hide yes)
+			(effects
+				(font
+					(size 1.27 1.27)
+				)
+			)
+		)
+		(property "Manufacturer" "Samsung Electro-Mechanics"
+			(at 50.8 101.6 0)
+			(hide yes)
+			(effects
+				(font
+					(size 1.27 1.27)
+				)
+			)
+		)
 		(pin "1"
 		)
@@
 			)
 		)
+		(property "MPN" "CL05B224KO5NNNC"
+			(at 101.6 101.6 0)
+			(hide yes)
+			(effects
+				(font
+					(size 1.27 1.27)
+				)
+			)
+		)
+		(property "LCSC" "C16772"
+			(at 101.6 101.6 0)
+			(hide yes)
+			(effects
+				(font
+					(size 1.27 1.27)
+				)
+			)
+		)
+		(property "Manufacturer" "Samsung Electro-Mechanics"
+			(at 101.6 101.6 0)
+			(hide yes)
+			(effects
+				(font
+					(size 1.27 1.27)
+				)
+			)
+		)
 		(pin "1"
 		)
@@
 			)
 		)
+		(property "MPN" "GRM0335C1H220JA01D"
+			(at 25.4 38.1 0)
+			(hide yes)
+			(effects
+				(font
+					(size 1.27 1.27)
+				)
+			)
+		)
+		(property "LCSC" "C76924"
+			(at 25.4 38.1 0)
+			(hide yes)
+			(effects
+				(font
+					(size 1.27 1.27)
+				)
+			)
+		)
+		(property "Manufacturer" "Murata"
+			(at 25.4 38.1 0)
+			(hide yes)
+			(effects
+				(font
+					(size 1.27 1.27)
+				)
+			)
+		)
 		(pin "1"
 		)
@@
 			)
 		)
+		(property "MPN" "GRM0335C1H220JA01D"
+			(at 35.56 38.1 0)
+			(hide yes)
+			(effects
+				(font
+					(size 1.27 1.27)
+				)
+			)
+		)
+		(property "LCSC" "C76924"
+			(at 35.56 38.1 0)
+			(hide yes)
+			(effects
+				(font
+					(size 1.27 1.27)
+				)
+			)
+		)
+		(property "Manufacturer" "Murata"
+			(at 35.56 38.1 0)
+			(hide yes)
+			(effects
+				(font
+					(size 1.27 1.27)
+				)
+			)
+		)
 		(pin "1"
 		)
@@
 			)
 		)
+		(property "MPN" "GRM0335C1H220JA01D"
+			(at 45.72 38.1 0)
+			(hide yes)
+			(effects
+				(font
+					(size 1.27 1.27)
+				)
+			)
+		)
+		(property "LCSC" "C76924"
+			(at 45.72 38.1 0)
+			(hide yes)
+			(effects
+				(font
+					(size 1.27 1.27)
+				)
+			)
+		)
+		(property "Manufacturer" "Murata"
+			(at 45.72 38.1 0)
+			(hide yes)
+			(effects
+				(font
+					(size 1.27 1.27)
+				)
+			)
+		)
 		(pin "1"
 		)
@@
 			(effects
 				(font
+					(size 1.27 1.27)
+				)
+			)
+		)
+		(property "MPN" "GRM0335C1H220JA01D"
+			(at 55.88 38.1 0)
+			(hide yes)
+			(effects
+				(font
+					(size 1.27 1.27)
+				)
+			)
+		)
+		(property "LCSC" "C76924"
+			(at 55.88 38.1 0)
+			(hide yes)
+			(effects
+				(font
+					(size 1.27 1.27)
+				)
+			)
+		)
+		(property "Manufacturer" "Murata"
+			(at 55.88 38.1 0)
+			(hide yes)
+			(effects
+				(font

Commit message: v2m-2: rename U4 footprint to Board:TI_TPD3F303_USON-8_DPV_2.1x1.6mm_P0.5mm (lib, PCB, schematic field - PM approved); lib synced to board copy, Board lib in fp-lib-table -> ${KIPRJMOD}; BOM.csv U4 package; jlc/BOM_JLC_v2.csv + new jlc/CPL_JLC_v2.csv (kicad-cli pos, both sides, excl. DNP). No U4 lib mismatch
Parts:
- U4: footprint Board:TI_TPD3F303_USON-8_1.45x1.45mm_P0.4mm -> Board:TI_TPD3F303_USON-8_DPV_2.1x1.6mm_P0.5mm
Changed lines of the file:
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@@
 			)
 		)
-		(property "Footprint" "Board:TI_TPD3F303_USON-8_1.45x1.45mm_P0.4mm"
+		(property "Footprint" "Board:TI_TPD3F303_USON-8_DPV_2.1x1.6mm_P0.5mm"
 			(at 49.53 53.34 0)
 			(hide yes)
